File: targetbunnybots.kicad_pcb (KiCad board)
At the start: 2 copper layers, 71.1 x 73.7 mm, 13 parts, among them J1 Conn_01x02, J2 Conn_01x05, J3 Conn_01x04, J4 Conn_01x04, J5 Raspberry_Pi_2_3, J6 Conn_01x06, J7 Conn_01x06, J8 Conn_01x03, J9 Conn_01x03

Commit message: Add files via upload
Parts:
- added ?: 1540Logo, Library:1540Logo, B.Cu at (167.8, 101.5)
- added H5: MountingHole, MountingHole:MountingHole_4mm, F.Cu at (114.3, 147.3)
- added H6: MountingHole, MountingHole:MountingHole_4mm, F.Cu at (139.7, 147.3)
- H2, H3: footprint MountingHole:MountingHole_2.5mm -> MountingHole:MountingHole_4mm
- J5: value Raspberry_Pi_2_3 -> Raspberry_Pi_Zero_W
- moved H3 70.7 mm to (139.7, 83.8)
- moved J2 6.86 mm to (122.0, 132.1)
- moved J1 5.47 mm to (114.3, 132.1)
- moved J4 2.54 mm to (121.9, 114.3)
- moved H2 2.51 mm to (114.3, 83.8)
Connections:
- net /LEDData renamed Net-(J7-Pin_6)
- net Net-(J3-Pin_1) renamed /Switch1
- net Net-(J3-Pin_2) renamed /Switch2
- net Net-(J3-Pin_3) renamed /Switch3
- net Net-(J3-Pin_4) renamed /Switch4
- J5 pad 17: unconnected-(J5-3V3-Pad17) -> +3.3V
- J5 pad 4: unconnected-(J5-5V-Pad4) -> +5V
Routing:
- net GND: track 16.8 -> 13.8 mm
- net +6V: track 13.2 -> 10.2 mm
Other:
- board text added: "GND"
- board text added: "Solder 5V Bridge On Supply!"
- board text added: "V"
- board text removed: "Power"
- board text removed: "V GND"
