File: targetbunnybots.kicad_sch (KiCad schematic)
At the start: 13 parts, among them J1 Conn_01x02, J2 Conn_01x05, J3 Conn_01x04, J4 Conn_01x04, J5 Raspberry_Pi_2_3, J6 Conn_01x06, J7 Conn_01x06, J8 Conn_01x03, J9 Conn_01x03

Commit message: Add files via upload
Parts:
- added H5, H6: MountingHole, MountingHole:MountingHole_5mm, symbol Mechanical:MountingHole
- H2: footprint MountingHole:MountingHole_2.5mm -> MountingHole:MountingHole_4mm
- H3: footprint MountingHole:MountingHole_2.5mm -> MountingHole:MountingHole_5mm
- J5: value Raspberry_Pi_2_3 -> Raspberry_Pi_Zero_W
Connections:
- net +3.3V: now also J5.17 (3V3)
- net +5V: now also J5.4 (5V)
- net Switch1: now reaches J3.1 (Pin_1), J5.19 (MOSI0/GPIO10)
- net Switch2: now reaches J3.2 (Pin_2), J5.21 (MISO0/GPIO9)
- net Switch3: now reaches J3.3 (Pin_3), J5.24 (~{CE0}/GPIO8)
- net Switch4: now reaches J3.4 (Pin_4), J5.26 (~{CE1}/GPIO7)
- net LEDData: no longer names the net of J7.6 (Pin_6), J8.2 (Pin_2)
Other:
- moved on the sheet: J8
